File: hardware/distance-ir-v3.kicad_pcb (KiCad board)
At the start: 2 copper layers, 0 parts

Commit message: pcb design
Parts:
- added C1: 100nF, kicad-libraries:C0603F, F.Cu at (114.6, 109.0)
- added C101: 10uF, kicad-libraries:C0805, F.Cu at (118.6, 105.5)
- added C102: 220pF, kicad-libraries:C0402F, F.Cu at (108.0, 107.1)
- added C103: 1uF, kicad-libraries:C0603F, F.Cu at (118.6, 107.0)
- added C104: 100nF, kicad-libraries:C0603F, F.Cu at (101.5, 110.1)
- added C2: 4,7uF, kicad-libraries:C0805E, F.Cu at (116.2, 109.0)
- added D101: blue, kicad-libraries:D0603F, F.Cu at (112.5, 117.5)
- added G***: LOGO, kicad-libraries:Logo_CoMCU, B.Cu at (112.5, 110.0)
- added G***: LOGO, kicad-libraries:Logo_31x31, F.Cu at (121.4, 110.0)
- added P101: CON-SENSOR2, kicad-libraries:CON-SENSOR2, F.Cu at (112.5, 100.0)
- added P102: DEBUG, kicad-libraries:DEBUG_PAD, F.Cu at (106.1, 106.4)
- added P103: BOOT, kicad-libraries:SolderJumper, F.Cu at (104.4, 106.4)
- added R101: 1k, kicad-libraries:R0603F, F.Cu at (109.5, 117.5)
- added RP1: 10k, kicad-libraries:0603X4, F.Cu at (112.5, 114.2)
- added RP101: 82, kicad-libraries:4X0402, F.Cu at (109.6, 107.1)
- added RP102: 3k9, kicad-libraries:0603X4, F.Cu at (109.0, 114.2)
- added U1: VL53L1, kicad-libraries:VL53L1, F.Cu at (112.5, 110.0)
- added U101: XMC1XXX, kicad-libraries:QFN24-4x4mm-0.5mm, F.Cu at (104.9, 110.0)
- added U103: DRILL, kicad-libraries:DRILL_NP, F.Cu at (102.5, 117.5)
- added U104: DRILL, kicad-libraries:DRILL_NP, F.Cu at (122.5, 102.5)
- added U105: DRILL, kicad-libraries:DRILL_NP, F.Cu at (122.5, 117.5)
- added U106: DRILL, kicad-libraries:DRILL_NP, F.Cu at (102.5, 102.5)
- added VAL: WEEE_7mm, kicad-libraries:WEEE_7mm, B.Cu at (105.3, 110.1)
- added VAL: CE_5mm, kicad-libraries:CE_5mm, B.Cu at (119.9, 110.0)
Routing:
- net VCC: track 0.00 -> 47.7 mm
- net GND: track 0.00 -> 26.4 mm, vias 0 -> 17
- net XSHUT: track 0.00 -> 10.6 mm, vias 0 -> 2
- net Net-(R101-Pad1): track 0.00 -> 8.05 mm, vias 0 -> 2
- net GPIO: track 0.00 -> 7.04 mm, vias 0 -> 2
- net SDA: track 2.47 -> 9.20 mm
- net SCL: track 2.60 -> 8.73 mm, vias 0 -> 2
- net S-CS: track 0.00 -> 4.80 mm
- net S-CLK: track 0.00 -> 3.97 mm
- net Net-(P101-Pad4): track 0.00 -> 3.59 mm
- net S-MISO: track 0.00 -> 3.31 mm
- net S-MOSI: track 0.00 -> 3.18 mm
- net Net-(P101-Pad5): track 0.00 -> 3.12 mm
- net Net-(C102-Pad2): track 0.00 -> 2.85 mm
- net Net-(P103-Pad2): track 0.00 -> 2.31 mm
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- added copper zone on F.Cu, net GND
- added copper zone on F.Cu, net VCC
Other:
- board outline added: 25 x 20 mm
- board text added: "Distance IR V3.0"
- board text added: "Status"
- board text added: "tinkerforge.com"

Commit message: added fiducial marks
Parts:
- added Fiducial_Mark: VAL**, kicad-libraries:Fiducial_Mark, F.Cu at (122.0, 107.0)
- added Fiducial_Mark: VAL**, kicad-libraries:Fiducial_Mark, F.Cu at (121.0, 113.0)
- added Fiducial_Mark: VAL**, kicad-libraries:Fiducial_Mark, F.Cu at (102.0, 107.0)
Changed lines of the file:
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@@
     (tracks 183)
     (zones 0)
-    (modules 24)
+    (modules 27)
     (nets 36)
   )
@@
   )
   (setup
-    (last_trace_width 0.25)
+    (last_trace_width 0.2)
     (user_trace_width 0.25)
     (user_trace_width 0.3)
@@
     (add_net XSHUT)
   )
+  (module kicad-libraries:Fiducial_Mark (layer F.Cu)
+    (at 122 107)
+    (attr smd)
+    (fp_text reference Fiducial_Mark (at 0 0) (layer F.SilkS) hide
+      (effects (font (size 0.127 0.127) (thickness 0.03302)))
+    )
+    (fp_text value VAL** (at 0 -0.29972) (layer F.SilkS) hide
+      (effects (font (size 0.127 0.127) (thickness 0.03302)))
+    )
+    (fp_circle (center 0 0) (end 1.15062 0) (layer Dwgs.User) (width 0.01016))
+    (pad 1 smd circle (at 0 0) (size 1.00076 1.00076) (layers F.Cu F.Paste F.Mask)
+      (clearance 0.65024))
+  )
+  (module kicad-libraries:Fiducial_Mark (layer F.Cu)
+    (at 121 113)
+    (attr smd)
+    (fp_text reference Fiducial_Mark (at 0 0) (layer F.SilkS) hide
+      (effects (font (size 0.127 0.127) (thickness 0.03302)))
+    )
+    (fp_text value VAL** (at 0 -0.29972) (layer F.SilkS) hide
+      (effects (font (size 0.127 0.127) (thickness 0.03302)))
+    )
+    (fp_circle (center 0 0) (end 1.15062 0) (layer Dwgs.User) (width 0.01016))
+    (pad 1 smd circle (at 0 0) (size 1.00076 1.00076) (layers F.Cu F.Paste F.Mask)
+      (clearance 0.65024))
+  )
+  (module kicad-libraries:Fiducial_Mark (layer F.Cu)
+    (at 102 107)
+    (attr smd)
+    (fp_text reference Fiducial_Mark (at 0 0) (layer F.SilkS) hide
+      (effects (font (size 0.127 0.127) (thickness 0.03302)))
+    )
+    (fp_text value VAL** (at 0 -0.29972) (layer F.SilkS) hide
+      (effects (font (size 0.127 0.127) (thickness 0.03302)))
+    )
+    (fp_circle (center 0 0) (end 1.15062 0) (layer Dwgs.User) (width 0.01016))
+    (pad 1 smd circle (at 0 0) (size 1.00076 1.00076) (layers F.Cu F.Paste F.Mask)
+      (clearance 0.65024))
+  )
   (module kicad-libraries:VL53L1 (layer F.Cu)

Commit message: changed sda and scl
Parts:
- moved Fiducial_Mark 6.04 mm to (118.5, 118.5)
Connections:
- RP102 pad 5: SCL -> SDA
- RP102 pad 8: SDA -> SCL
- U1 pad 10: SDA -> SCL
- U1 pad 9: SCL -> SDA
Routing:
- net SDA: track 9.20 -> 10.9 mm
- net SCL: track 8.73 -> 8.52 mm, vias 2 -> 0
Changed lines of the file:
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@@
     (thickness 1.6)
     (drawings 12)
-    (tracks 183)
+    (tracks 178)
     (zones 0)
     (modules 27)
@@
   )
   (setup
-    (last_trace_width 0.2)
+    (last_trace_width 0.25)
     (user_trace_width 0.25)
     (user_trace_width 0.3)
@@
   )
   (module kicad-libraries:Fiducial_Mark (layer F.Cu)
-    (at 121 113)
+    (at 118.5 118.5)
     (attr smd)
     (fp_text reference Fiducial_Mark (at 0 0) (layer F.SilkS) hide
@@
       (net 4 VCC))
     (pad 10 smd rect (at 0.8 -0.8 90) (size 0.5 0.5) (layers F.Cu F.Paste F.Mask)
+      (net 3 SCL))
+    (pad 9 smd rect (at 0 -0.8 90) (size 0.5 0.5) (layers F.Cu F.Paste F.Mask)
       (net 2 SDA))
-    (pad 9 smd rect (at 0 -0.8 90) (size 0.5 0.5) (layers F.Cu F.Paste F.Mask)
-      (net 3 SCL))
     (pad 8 smd rect (at -0.8 -0.8 90) (size 0.5 0.5) (layers F.Cu F.Paste F.Mask)
       (net 24 "Net-(U1-Pad8)"))
@@
       (net 4 VCC))
     (pad 5 smd rect (at -1.19888 0.8509 180) (size 0.44958 0.89916) (layers F.Cu F.Paste F.Mask)
-      (net 3 SCL))
+      (net 2 SDA))
     (pad 6 smd rect (at -0.39878 0.8509 180) (size 0.44958 0.89916) (layers F.Cu F.Paste F.Mask)
       (net 22 "Net-(RP102-Pad6)"))
@@
       (net 23 "Net-(RP102-Pad7)"))
     (pad 8 smd rect (at 1.19888 0.8509 180) (size 0.44958 0.89916) (layers F.Cu F.Paste F.Mask)
-      (net 2 SDA))
+      (net 3 SCL))
     (model Resistors_SMD/R_4x0603.wrl
       (at (xyz 0 0 0))
@@
   (segment (start 117.85 107.44) (end 117.82499 107.44) (width 0.5) (layer F.Cu) (net 1))
   (segment (start 117.82499 107.44) (end 117.764999 107.499991) (width 0.5) (layer F.Cu) (net 1))
-  (segment (start 107.32633 113.3491) (end 107.80112 113.3491) (width 0.25) (layer F.Cu) (net 2))
-  (segment (start 105.65 112.775) (end 106.2241 113.3491) (width 0.25) (layer F.Cu) (net 2))
-  (segment (start 106.2241 113.3491) (end 107.32633 113.3491) (width 0.25) (layer F.Cu) (net 2))
-  (segment (start 105.65 112.025) (end 105.65 112.775) (width 0.25) (layer F.Cu) (net 2))
-  (segment (start 107.80112 112.59888) (end 111.2 109.2) (width 0.25) (layer F.Cu) (net 2))
-  (segment (start 111.2 109.2) (end 111.7 109.2) (width 0.25) (layer F.Cu) (net 2))
-  (segment (start 107.80112 113.3491) (end 107.80112 112.59888) (width 0.25) (layer F.Cu) (net 2))
-  (via (at 109 112.2) (size 0.55) (drill 0.25) (layers F.Cu B.Cu) (net 3))
-  (segment (start 111.2 110) (end 111.7 110) (width 0.25) (layer F.Cu) (net 3))
-  (segment (start 110.19888 111.00112) (end 111.2 110) (width 0.25) (layer F.Cu) (net 3))
-  (segment (start 110.19888 113.3491) (end 110.19888 111.00112) (width 0.25) (layer F.Cu) (net 3))
-  (segment (start 110.19888 112.79888) (end 110.19888 113.3491) (width 0.25) (layer F.Cu) (net 3))
-  (segment (start 109.6 112.2) (end 110.19888 112.79888) (width 0.25) (layer F.Cu) (net 3))
-  (segment (start 109 112.2) (end 109.6 112.2) (width 0.25) (layer F.Cu) (net 3))
-  (segment (start 109 112.2) (end 108.232082 111.432082) (width 0.25) (layer B.Cu) (net 3))
-  (via (at 108.178978 111.432082) (size 0.55) (drill 0.25) (layers F.Cu B.Cu) (net 3))
-  (segment (start 108.232082 111.432082) (end 108.178978 111.432082) (width 0.25) (layer B.Cu) (net 3))
-  (segment (start 106.925 111.25) (end 107.996896 111.25) (width 0.25) (layer F.Cu) (net 3))
-  (segment (start 107.996896 111.25) (end 108.178978 111.432082) (width 0.25) (layer F.Cu) (net 3))
+  (segment (start 107.80112 112.59888) (end 111.2 109.2) (width 0.25) (layer F.Cu) (net 3))
+  (segment (start 111.2 109.2) (end 111.7 109.2) (width 0.25) (layer F.Cu) (net 3))
+  (segment (start 107.80112 113.3491) (end 107.80112 112.59888) (width 0.25) (layer F.Cu) (net 3))
+  (segment (start 111.2 110) (end 111.7 110) (width 0.25) (layer F.Cu) (net 2))
+  (segment (start 110.19888 111.00112) (end 111.2 110) (width 0.25) (layer F.Cu) (net 2))
+  (segment (start 110.19888 113.3491) (end 110.19888 111.00112) (width 0.25) (layer F.Cu) (net 2))
+  (segment (start 107.075 114.2) (end 105.65 112.775) (width 0.25) (layer F.Cu) (net 2))
+  (segment (start 110.04756 114.2) (end 107.075 114.2) (width 0.25) (layer F.Cu) (net 2))
+  (segment (start 105.65 112.775) (end 105.65 112.025) (width 0.25) (layer F.Cu) (net 2))
+  (segment (start 110.19888 114.04868) (end 110.04756 114.2) (width 0.25) (layer F.Cu) (net 2))
+  (segment (start 110.19888 113.3491) (end 110.19888 114.04868) (width 0.25) (layer F.Cu) (net 2))
+  (segment (start 107.80112 112.60112) (end 107.80112 113.3491) (width 0.25) (layer F.Cu) (net 3))
+  (segment (start 106.925 111.725) (end 107.80112 112.60112) (width 0.25) (layer F.Cu) (net 3))
+  (segment (start 106.925 111.25) (end 106.925 111.725) (width 0.25) (layer F.Cu) (net 3))
   (segment (start 114.828499 108.021501) (end 114.6 108.25) (width 0.8) (layer F.Cu) (net 4))
   (segment (start 116.179399 108.021501) (end 114.828499 108.021501) (width 0.8) (layer F.Cu) (net 4))

Commit message: changed footprint for incoming capacitors
Parts:
- C101: footprint kicad-libraries:C0805 -> tinkerforge:C0805E
- C103: footprint kicad-libraries:C0603F -> tinkerforge:C0603F
Changed lines of the file:
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@@
-(kicad_pcb (version 20171130) (host pcbnew 5.1.5+dfsg1-2build2)
+(kicad_pcb (version 20171130) (host pcbnew "(5.1.4)-1")
   (general
     (thickness 1.6)
@@
   )
   (setup
-    (last_trace_width 0.25)
+    (last_trace_width 0.2)
     (user_trace_width 0.25)
     (user_trace_width 0.3)
@@
     (aux_axis_origin 100 100)
     (grid_origin 100 100)
-    (visible_elements FFFEFF7F)
+    (visible_elements 7FFFFFFF)
     (pcbplotparams
       (layerselection 0x00010_00000000)
@@
     )
   )
-  (module kicad-libraries:C0805 (layer F.Cu)
-    (at 118.6 105.5)
-    (attr smd)
-    (fp_text reference C101 (at 0 0.3) (layer F.Fab)
-      (effects (font (size 0.2 0.2) (thickness 0.05)))
-    )
-    (fp_text value 10uF (at 0 -0.2) (layer F.Fab)
-      (effects (font (size 0.2 0.2) (thickness 0.05)))
-    )
-    (fp_line (start -1.651 -0.8001) (end -1.651 0.8001) (layer F.Fab) (width 0.001))
-    (fp_line (start -1.651 0.8001) (end 1.651 0.8001) (layer F.Fab) (width 0.001))
-    (fp_line (start 1.651 0.8001) (end 1.651 -0.8001) (layer F.Fab) (width 0.001))
-    (fp_line (start 1.651 -0.8001) (end -1.651 -0.8001) (layer F.Fab) (width 0.001))
-    (pad 1 smd rect (at -1.00076 0) (size 1.00076 1.24968) (layers F.Cu F.Paste F.Mask)
-      (net 1 GND) (clearance 0.14986))
-    (pad 2 smd rect (at 1.00076 0) (size 1.00076 1.24968) (layers F.Cu F.Paste F.Mask)
-      (net 4 VCC) (clearance 0.14986))
-    (model Capacitors_SMD/C_0805.wrl
-      (at (xyz 0 0 0))
-      (scale (xyz 1 1 1))
-      (rotate (xyz 0 0 0))
-    )
-  )
   (module kicad-libraries:C0402F (layer F.Cu)
     (at 108 107.1 90)
@@
       (net 1 GND))
     (model Capacitors_SMD/C_0402.wrl
-      (at (xyz 0 0 0))
-      (scale (xyz 1 1 1))
-      (rotate (xyz 0 0 0))
-    )
-  )
-  (module kicad-libraries:C0603F (layer F.Cu)
-    (at 118.6 107)
-    (attr smd)
-    (fp_text reference C103 (at 0.05 0.225) (layer F.Fab)
-      (effects (font (size 0.2 0.2) (thickness 0.05)))
-    )
-    (fp_text value 1uF (at 0.05 -0.375) (layer F.Fab)
-      (effects (font (size 0.2 0.2) (thickness 0.05)))
-    )
-    (fp_line (start -1.45034 -0.65024) (end 1.45034 -0.65024) (layer F.Fab) (width 0.001))
-    (fp_line (start 1.45034 -0.65024) (end 1.45034 0.65024) (layer F.Fab) (width 0.001))
-    (fp_line (start 1.45034 0.65024) (end -1.45034 0.65024) (layer F.Fab) (width 0.001))
-    (fp_line (start -1.45034 0.65024) (end -1.45034 -0.65024) (layer F.Fab) (width 0.001))
-    (pad 1 smd rect (at -0.75 0) (size 0.9 0.9) (layers F.Cu F.Paste F.Mask)
-      (net 1 GND))
-    (pad 2 smd rect (at 0.75 0) (size 0.9 0.9) (layers F.Cu F.Paste F.Mask)
-      (net 4 VCC))
-    (model Capacitors_SMD/C_0603.wrl
       (at (xyz 0 0 0))
       (scale (xyz 1 1 1))
@@
     (pad "" np_thru_hole circle (at 0 0) (size 2.99974 2.99974) (drill 2.99974) (layers *.Cu *.Mask F.SilkS)
       (clearance 0.89916))
+  )
+  (module tinkerforge:C0805E (layer F.Cu)
+    (at 118.6 105.5)
+    (attr smd)
+    (fp_text reference C101 (at 0 0.2) (layer F.Fab)
+      (effects (font (size 0.2 0.2) (thickness 0.05)))
+    )
+    (fp_text value 10uF (at 0 -0.4) (layer F.Fab)
+      (effects (font (size 0.2 0.2) (thickness 0.05)))
+    )
+    (fp_line (start -1.651 -0.8001) (end -1.651 0.8001) (layer F.Fab) (width 0.001))
+    (fp_line (start -1.651 0.8001) (end 1.651 0.8001) (layer F.Fab) (width 0.001))
+    (fp_line (start 1.651 0.8001) (end 1.651 -0.8001) (layer F.Fab) (width 0.001))
+    (fp_line (start 1.651 -0.8001) (end -1.651 -0.8001) (layer F.Fab) (width 0.001))
+    (pad 1 smd rect (at -0.95 0) (size 1.3 1.5) (layers F.Cu F.Paste F.Mask)
+      (net 1 GND) (clearance 0.14986))
+    (pad 2 smd rect (at 0.95 0) (size 1.3 1.5) (layers F.Cu F.Paste F.Mask)
+      (net 4 VCC) (clearance 0.14986))
+    (model Capacitors_SMD/C_0805.wrl
+      (at (xyz 0 0 0))
+      (scale (xyz 1 1 1))
+      (rotate (xyz 0 0 0))
+    )
+  )
+  (module tinkerforge:C0603F (layer F.Cu)
+    (at 118.6 107)
+    (attr smd)
+    (fp_text reference C103 (at 0.05 0.225) (layer F.Fab)
+      (effects (font (size 0.2 0.2) (thickness 0.05)))
+    )
+    (fp_text value 1uF (at 0.05 -0.375) (layer F.Fab)
+      (effects (font (size 0.2 0.2) (thickness 0.05)))
+    )
+    (fp_line (start -1.45034 -0.65024) (end 1.45034 -0.65024) (layer F.Fab) (width 0.001))
+    (fp_line (start 1.45034 -0.65024) (end 1.45034 0.65024) (layer F.Fab) (width 0.001))
+    (fp_line (start 1.45034 0.65024) (end -1.45034 0.65024) (layer F.Fab) (width 0.001))
+    (fp_line (start -1.45034 0.65024) (end -1.45034 -0.65024) (layer F.Fab) (width 0.001))
+    (pad 1 smd rect (at -0.75 0) (size 0.9 0.9) (layers F.Cu F.Paste F.Mask)
+      (net 1 GND))
+    (pad 2 smd rect (at 0.75 0) (size 0.9 0.9) (layers F.Cu F.Paste F.Mask)
+      (net 4 VCC))
+    (model Capacitors_SMD/C_0603.wrl
+      (at (xyz 0 0 0))
+      (scale (xyz 1 1 1))
+      (rotate (xyz 0 0 0))
+    )
   )
   (gr_text tinkerforge.com (at 123.7 110 90) (layer F.SilkS)
@@
   (segment (start 117.85 107.44) (end 117.82499 107.44) (width 0.5) (layer F.Cu) (net 1))
   (segment (start 117.82499 107.44) (end 117.764999 107.499991) (width 0.5) (layer F.Cu) (net 1))
-  (segment (start 107.80112 112.59888) (end 111.2 109.2) (width 0.25) (layer F.Cu) (net 3))
-  (segment (start 111.2 109.2) (end 111.7 109.2) (width 0.25) (layer F.Cu) (net 3))
-  (segment (start 107.80112 113.3491) (end 107.80112 112.59888) (width 0.25) (layer F.Cu) (net 3))
   (segment (start 111.2 110) (end 111.7 110) (width 0.25) (layer F.Cu) (net 2))
   (segment (start 110.19888 111.00112) (end 111.2 110) (width 0.25) (layer F.Cu) (net 2))
@@
   (segment (start 110.19888 114.04868) (end 110.04756 114.2) (width 0.25) (layer F.Cu) (net 2))
   (segment (start 110.19888 113.3491) (end 110.19888 114.04868) (width 0.25) (layer F.Cu) (net 2))
+  (segment (start 107.80112 112.59888) (end 111.2 109.2) (width 0.25) (layer F.Cu) (net 3))
+  (segment (start 111.2 109.2) (end 111.7 109.2) (width 0.25) (layer F.Cu) (net 3))
+  (segment (start 107.80112 113.3491) (end 107.80112 112.59888) (width 0.25) (layer F.Cu) (net 3))
   (segment (start 107.80112 112.60112) (end 107.80112 113.3491) (width 0.25) (layer F.Cu) (net 3))
   (segment (start 106.925 111.725) (end 107.80112 112.60112) (width 0.25) (layer F.Cu) (net 3))
